Commit message: Fix mesh and controller paths in urdf
Co-Authored-By: Claude Opus 4.8 <noreply@anthropic.com>

File: urdf/5dof_arm.urdf (robot description, URDF)
Before this commit: robot 5dof_arm, 7 links, 6 joints
Links:
- link base_link: geometry collision mesh filename=package://arm_5dof/meshes/base_link.stl scale=0.001 0.001 0.001; visual mesh filename=package://arm_5dof/meshes/base_link.stl scale=0.001 0.001 0.001
- link link0: geometry collision mesh filename=package://arm_5dof/meshes/link0.stl scale=0.001 0.001 0.001; visual mesh filename=package://arm_5dof/meshes/link0.stl scale=0.001 0.001 0.001
- link link1: geometry collision mesh filename=package://arm_5dof/meshes/link1.stl scale=0.001 0.001 0.001; visual mesh filename=package://arm_5dof/meshes/link1.stl scale=0.001 0.001 0.001
- link link2: geometry collision mesh filename=package://arm_5dof/meshes/link2.stl scale=0.001 0.001 0.001; visual mesh filename=package://arm_5dof/meshes/link2.stl scale=0.001 0.001 0.001
- link link3: geometry collision mesh filename=package://arm_5dof/meshes/link3.stl scale=0.001 0.001 0.001; visual mesh filename=package://arm_5dof/meshes/link3.stl scale=0.001 0.001 0.001
- link link4: geometry collision mesh filename=package://arm_5dof/meshes/link4.stl scale=0.001 0.001 0.001; visual mesh filename=package://arm_5dof/meshes/link4.stl scale=0.001 0.001 0.001
